File: hardware/triptech.kicad_sch (KiCad schematic)
At the start: 0 parts

Commit message: PCB Assembledish Design checks next
Parts:
- added H1, H2, H3, H4, H5: MountingHole, MountingHole:MountingHole_3.2mm_M3, symbol Mechanical:MountingHole
