File: hardware/audio.kicad_sch (KiCad schematic)
At the start: 51 parts, among them J10 Earth, J4 NCJ6FA-H-0, J5 NCJ6FA-H-0, J6 Conn_01x04_Pin, J7 Earth, J8 NCJ6FA-H-0, J9 NCJ6FA-H-0, U5 THAT1246, U6 THAT1246, U7 THAT1646, U8 THAT1646

Commit message: PCB rev 1
Changed lines of the file:
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@@
 	)
 	(junction
+		(at 31.75 120.65)
+		(diameter 0)
+		(color 0 0 0 0)
+	)
+	(junction
 		(at 241.3 36.83)
 		(diameter 0)
@@
 	(wire
 		(pts
+			(xy 22.86 125.73) (xy 22.86 120.65)
+		)
+		(stroke
+			(width 0)
+			(type default)
+		)
+	)
+	(wire
+		(pts
 			(xy 184.15 104.14) (xy 195.58 104.14)
 		)
@@
 	(wire
 		(pts
+			(xy 31.75 120.65) (xy 31.75 110.49)
+		)
+		(stroke
+			(width 0)
+			(type default)
+		)
+	)
+	(wire
+		(pts
 			(xy 48.26 110.49) (xy 43.18 110.49)
 		)
@@
 	(wire
 		(pts
+			(xy 22.86 120.65) (xy 31.75 120.65)
+		)
+		(stroke
+			(width 0)
+			(type default)
+		)
+	)
+	(wire
+		(pts
 			(xy 34.29 44.45) (xy 48.26 44.45)
 		)
@@
 	(wire
 		(pts
-			(xy 31.75 121.92) (xy 31.75 110.49)
+			(xy 31.75 121.92) (xy 31.75 120.65)
 		)
 		(stroke
@@
 					(unit 1)
 				)
+			)
+		)
+	)
+	(symbol
+		(lib_id "power:PWR_FLAG")
+		(at 22.86 125.73 0)
+		(mirror x)
+		(unit 1)
+		(exclude_from_sim no)
+		(in_bom yes)
+		(on_board yes)
+		(dnp no)
+		(property "Reference" "#FLG05"
+			(at 22.86 127.635 0)
+			(effects
+				(font
+					(size 1.27 1.27)
+				)
+				(hide yes)
+			)
+		)
+		(property "Value" "PWR_FLAG_Earth"
+			(at 22.86 130.81 0)
+			(effects
+				(font
+					(size 1.27 1.27)
+				)
+			)
+		)
+		(property "Footprint" ""
+			(at 22.86 125.73 0)
+			(effects
+				(font
+					(size 1.27 1.27)
+				)
+				(hide yes)
+			)
+		)
+		(property "Datasheet" "~"
+			(at 22.86 125.73 0)
+			(effects
+				(font
+					(size 1.27 1.27)
+				)
+				(hide yes)
+			)
+		)
+		(property "Description" "Special symbol for telling ERC where power comes from"
+			(at 22.86 125.73 0)
+			(effects
+				(font
+					(size 1.27 1.27)
+				)
+				(hide yes)
+			)
+		)
+		(pin "1"
+		)
+		(instances
+			(project "triptech"
+				(path "/55cca6a8-30da-4c13-b2f2-a01401e2b54c/a1b2c3d4-7777-4000-8000-000000000007"
+					(reference "#FLG05")
+					(unit 1)
+				)
